File: TekDaqc_RevE/TekDAQC_RevE.kicad_pcb (KiCad board)
At the start: 2 copper layers, 194.9 x 241.1 mm, 443 parts, among them T1 4POLE_PLUGIN_TERMINAL_SIDE, T10 6POLE_PLUGIN_TERMINAL_SIDE, T11 6POLE_PLUGIN_TERMINAL_SIDE, T12 6POLE_PLUGIN_TERMINAL_SIDE, T13 4POLE_PLUGIN_TERMINAL_SIDE, T14 4POLE_PLUGIN_TERMINAL_SIDE, T15 4POLE_PLUGIN_TERMINAL_SIDE, T16 4POLE_PLUGIN_TERMINAL_SIDE, T17 8POLE_PLUGIN_TERMINAL_TOP, T18 8POLE_PLUGIN_TERMINAL_TOP, T19 8POLE_PLUGIN_TERMINAL_TOP, T2 4POLE_PLUGIN_TERMINAL_SIDE, T20 8POLE_PLUGIN_TERMINAL_TOP, T21 6POLE_PLUGIN_TERMINAL_TOP, T22 6POLE_PLUGIN_TERMINAL_TOP, T23 6POLE_PLUGIN_TERMINAL_TOP, T24 6POLE_PLUGIN_TERMINAL_TOP, T3 4POLE_PLUGIN_TERMINAL_SIDE, T4 4POLE_PLUGIN_TERMINAL_SIDE, T5 8POLE_PLUGIN_TERMINAL_SIDE, T6 8POLE_PLUGIN_TERMINAL_SIDE, T7 8POLE_PLUGIN_TERMINAL_SIDE, T8 8POLE_PLUGIN_TERMINAL_SIDE, T9 6POLE_PLUGIN_TERMINAL_SIDE, U1 SPIDER-TLE7232GS, U10 ADS1256, U11 STM32_CARRIERF407IGT6, U12 LM7805-T0220, U13 ISO7241CDW, U14 LM1086-3.3, U15 LM35, U16 VALOR_PM6045, U18 7404MTCX, U2 CD74HC154M96, U3 SPIDER-TLE7232GS, U4 CD74HC154M96, U5 MODULAR_JACK, U6 MCP2551_SOIC, U7 LTC6655BHLS8-2.5, U8 ISO7241CDW, U9 TF-SD, Y1 HCM49-7.680MABJ-UT

Commit message: current tekdaqc unmodified
Parts:
- added D31: B, CHIPLED_0805, F.Cu at (74.7, 155.5)
- added D32: B, CHIPLED_0805, F.Cu at (74.7, 140.1)
- added D33: B, CHIPLED_0805, F.Cu at (74.7, 124.5)
- added D34: B, CHIPLED_0805, F.Cu at (74.7, 112.9)
- added D35: B, CHIPLED_0805, F.Cu at (74.7, 166.9)
- added D36: B, CHIPLED_0805, F.Cu at (74.7, 147.6)
- added D37: B, CHIPLED_0805, F.Cu at (74.7, 135.9)
- added D38: B, CHIPLED_0805, F.Cu at (74.7, 120.7)
- added D52: B, CHIPLED_0805, F.Cu at (74.7, 159.3)
- added D53: B, CHIPLED_0805, F.Cu at (74.7, 144.0)
- added D54: B, CHIPLED_0805, F.Cu at (74.7, 128.3)
- added D55: B, CHIPLED_0805, F.Cu at (74.7, 109.0)
- added D58: B, CHIPLED_0805, F.Cu at (74.7, 163.1)
- added D59: B, CHIPLED_0805, F.Cu at (74.7, 151.4)
- added D60: B, CHIPLED_0805, F.Cu at (74.7, 132.1)
- added D61: B, CHIPLED_0805, F.Cu at (74.7, 116.7)
- added R51: 1M, M0805, F.Cu at (74.7, 157.4)
- added R52: 1M, M0805, F.Cu at (74.7, 142.0)
- added R53: 1M, M0805, F.Cu at (74.7, 126.4)
- added R54: 1M, M0805, F.Cu at (74.7, 114.8)
- added R59: 1M, M0805, F.Cu at (74.7, 168.7)
- added R60: 1M, M0805, F.Cu at (74.7, 149.5)
- added R61: 1M, M0805, F.Cu at (74.7, 137.8)
- added R62: 1M, M0805, F.Cu at (74.7, 122.6)
- added R89: 1M, M0805, F.Cu at (74.7, 161.2)
- added R90: 1M, M0805, F.Cu at (74.7, 145.9)
- added R91: 1M, M0805, F.Cu at (74.7, 130.2)
- added R92: 1M, M0805, F.Cu at (74.7, 111.0)
- added R95: 1M, M0805, F.Cu at (74.7, 165.0)
- added R96: 1M, M0805, F.Cu at (74.7, 153.4)
- added R97: 1M, M0805, F.Cu at (74.7, 134.0)
- added R98: 1M, M0805, F.Cu at (74.7, 118.6)
- JP2, JP3: footprint PINHEAD_1X10 -> 1X10
- R100, R101, R102, R107, R108, R109, R110, R63, R64, R65, R66, R71, R72, R73, R74, R99: value 1K -> 442; footprint RESISTOR_M0805 -> M0805
- T1, T2, T3, T4: footprint TEKDAQC_4POLE_3.5MM_TERMINAL_SIDE -> 4POLE_3.5MM_TERMINAL_SIDE
- T13, T14, T15, T16: value 4POLE_PLUGIN_TERMINAL_SIDE -> 4POLE_PLUGIN_TERMINAL_TOP; footprint TEKDAQC_4POLE_3.5MM_TERMINAL_TOP -> 4POLE_3.5MM_TERMINAL_TOP
- U1, U3: footprint SPIDER_TLE7232GS_SSOP24 -> SSOP24
Connections:
- R100 pad 2: T15.2 -> /TekDAQC_RevE_DO.sch/N$138
- R101 pad 2: T14.2 -> /TekDAQC_RevE_DO.sch/N$136
- R102 pad 2: T13.2 -> /TekDAQC_RevE_DO.sch/N$127
- R107 pad 2: T16.4 -> /TekDAQC_RevE_DO.sch/N$141
- R108 pad 2: T15.4 -> /TekDAQC_RevE_DO.sch/N$139
- R109 pad 2: T14.4 -> /TekDAQC_RevE_DO.sch/N$137
- R110 pad 2: T13.4 -> /TekDAQC_RevE_DO.sch/N$135
- R63 pad 2: T12.2 -> /TekDAQC_RevE_DO.sch/N$98
- R64 pad 2: T11.2 -> /TekDAQC_RevE_DO.sch/N$122
- R65 pad 2: T10.2 -> /TekDAQC_RevE_DO.sch/N$120
- R66 pad 2: T9.2 -> /TekDAQC_RevE_DO.sch/N$109
- R71 pad 2: T12.4 -> /TekDAQC_RevE_DO.sch/N$99
- R72 pad 2: T11.4 -> /TekDAQC_RevE_DO.sch/N$123
- R73 pad 2: T10.4 -> /TekDAQC_RevE_DO.sch/N$121
- R74 pad 2: T9.4 -> /TekDAQC_RevE_DO.sch/N$119
- R99 pad 2: T16.2 -> /TekDAQC_RevE_DO.sch/N$140
- U11 pad PC14: Net-(U11-PadPC14) -> GPI15
- U11 pad PH0: Net-(U11-PadPH0) -> GPI4
- U11 pad PH3: GPI4 -> Net-(U11-PadPH3)
- U11 pad PH5: GPI15 -> Net-(U11-PadPH5)
Routing:
- net GPI15: track 80.2 -> 39.3 mm, vias 3 -> 1
- net GPI4: track 76.2 -> 57.9 mm, vias 3 -> 1
- net T14.4: track 63.1 -> 57.4 mm
- net /TekDAQC_RevE_DO.sch/N$136: track 0.00 -> 5.32 mm
- net /TekDAQC_RevE_DO.sch/N$123: track 0.00 -> 5.26 mm
- net /TekDAQC_RevE_DO.sch/N$137: track 0.00 -> 5.22 mm
- net /TekDAQC_RevE_DO.sch/N$135: track 0.00 -> 5.05 mm
- net /TekDAQC_RevE_DO.sch/N$139: track 0.00 -> 5.03 mm
- net /TekDAQC_RevE_DO.sch/N$127: track 0.00 -> 5.01 mm
- net /TekDAQC_RevE_DO.sch/N$119: track 0.00 -> 4.98 mm
- net /TekDAQC_RevE_DO.sch/N$120: track 0.00 -> 4.90 mm
- net /TekDAQC_RevE_DO.sch/N$122: track 0.00 -> 4.90 mm
- net /TekDAQC_RevE_DO.sch/N$138: track 0.00 -> 4.89 mm
- net /TekDAQC_RevE_DO.sch/N$141: track 0.00 -> 4.89 mm
- net /TekDAQC_RevE_DO.sch/N$140: track 0.00 -> 4.89 mm
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Other:
- net class Default: trace_width 1.016 -> 0.508
- board text removed: "1. Printed circuit board made from 370HR epoxy laminate or equivilant with 1 oz. copper plating and 125 mil thickness."
