File: TekDaqc_RevE/TekDAQC_RevE.sch (KiCad schematic (older format))
At the start: 38 parts, among them U11 STM32_CARRIERF407IGT6, U5 MODULAR_JACK, U6 MCP2551_SOIC, U9 TF-SD

Commit message: current tekdaqc unmodified
Connections:
- net GPI15: now also U11.PC14; no longer U11.PH5
- net GPI4: now also U11.PH0; no longer U11.PH3
Changed lines of the file:
@@
 EESchema Schematic File Version 2
-LIBS:TekDAQC_RevE-rescue
-LIBS:power
-LIBS:device
-LIBS:transistors
-LIBS:conn
-LIBS:linear
-LIBS:regul
-LIBS:74xx
-LIBS:cmos4000
-LIBS:adc-dac
-LIBS:memory
-LIBS:xilinx
-LIBS:microcontrollers
-LIBS:dsp
-LIBS:microchip
-LIBS:analog_switches
-LIBS:motorola
-LIBS:texas
-LIBS:intel
-LIBS:audio
-LIBS:interface
-LIBS:digital-audio
-LIBS:philips
-LIBS:display
-LIBS:cypress
-LIBS:siliconi
-LIBS:opto
-LIBS:atmel
-LIBS:contrib
-LIBS:valves
 LIBS:TekDAQC_RevE
 LIBS:TekDAQC_RevE-cache
@@
 Text GLabel 1850 4650 0    60   Input ~ 0
 GPI16
-Text GLabel 4650 8655 3    60   Input ~ 0
+Text GLabel 1845 4750 0    60   Input ~ 0
 GPI4
 Text GLabel 1550 4950 0    60   Input ~ 0
@@
 	2050 4150 1850 4150
 Wire Wire Line
-	4650 8150 4650 8655
+	2050 4750 1845 4750
 Wire Wire Line
 	2050 5650 1850 5650
@@
 NoConn ~ 11850 7600
 NoConn ~ 11850 7500
-Text GLabel 5050 8650 3    60   Input ~ 0
+Text GLabel 1850 3950 0    60   Input ~ 0
 GPI15
 Wire Wire Line
-	5050 8650 5050 8150
-Text Label 5050 8150 3    10   ~ 0
+	1850 3950 2050 3950
+Text Label 2040 3950 2    10   ~ 0
 GPI15
 Text Label 7450 7150 0    10   ~ 0
@@
 Wire Wire Line
 	1650 5350 2050 5350
-NoConn ~ 2050 3950
-NoConn ~ 2050 4750
+NoConn ~ 4650 8150
+NoConn ~ 5050 8150
 $EndSCHEMATC
