File: TekDaqc_RevE/TekDAQC_RevE_DO.sch (KiCad schematic (older format))
At the start: 61 parts, among them T1 4POLE_PLUGIN_TERMINAL_SIDE, T10 6POLE_PLUGIN_TERMINAL_SIDE, T11 6POLE_PLUGIN_TERMINAL_SIDE, T12 6POLE_PLUGIN_TERMINAL_SIDE, T13 4POLE_PLUGIN_TERMINAL_SIDE, T14 4POLE_PLUGIN_TERMINAL_SIDE, T15 4POLE_PLUGIN_TERMINAL_SIDE, T16 4POLE_PLUGIN_TERMINAL_SIDE, T17 8POLE_PLUGIN_TERMINAL_TOP, T18 8POLE_PLUGIN_TERMINAL_TOP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

Commit message: current tekdaqc unmodified
Parts:
- removed T13, T14, T15, T16: 4POLE_PLUGIN_TERMINAL_SIDE, TekDAQC_RevE:TEKDAQC_4POLE_3.5MM_TERMINAL_SIDE, symbol TENKIV-TEKDAQC_4POLE_PLUGIN_TERMINAL_SIDE
- added D31, D32, D33, D34, D35, D36, D37, D38, D52, D53, D54, D55, D58, D59, D60, D61: B, TekDAQC_RevC:LED_CHIPLED_0805, symbol LED_LEDCHIPLED_0805
- added R51, R52, R53, R54, R59, R60, R61, R62, R89, R90, R91, R92, R95, R96, R97, R98: 1M, TekDAQC_RevC:RESISTOR_M0805, symbol RESISTOR_R-US_M0805
- added T13, T14, T15, T16: 4POLE_PLUGIN_TERMINAL_TOP, TENKIV TEKDAQC_4POLE_3.5MM_TERMINAL_TOP, symbol TENKIV-TEKDAQC_4POLE_PLUGIN_TERMINAL_TOP
- R100, R101, R102, R107, R108, R109, R110, R63, R64, R65, R66, R71, R72, R73, R74, R99: value 1K -> 442; footprint RESISTOR_M0805 -> TekDAQC_RevC:RESISTOR_M0805
- T1, T2, T3, T4: footprint TekDAQC_RevE:TEKDAQC_4POLE_3.5MM_TERMINAL_SIDE -> TENKIV TEKDAQC_4POLE_3.5MM_TERMINAL_SIDE
Connections:
- net N$77: now also T13.1, T13.3, T14.1, T14.3, T15.1, T15.3, T16.1, T16.3
- net T10.2: now also D33.C, R53.2; no longer R65.2
- net T10.4: now also D37.C, R61.2; no longer R73.2
- net T11.2: now also D32.C, R52.2; no longer R64.2
- net T11.4: now also D36.C, R60.2; no longer R72.2
- net T12.2: now also D31.C, R51.2; no longer R63.2
- net T12.4: now also D35.C, R59.2; no longer R71.2
- net T13.2: now also D55.C, R92.2, T16.2; no longer R102.2
- net T13.4: now also D61.C, R98.2, T16.4; no longer R110.2
- net T14.2: now also D54.C, R91.2, T15.2; no longer R101.2
- net T14.4: now also D60.C, R97.2, T15.4; no longer R109.2
- net T15.2: now also D53.C, R90.2, T14.2; no longer R100.2
- net T15.4: now also D59.C, R96.2, T14.4; no longer R108.2
- net T16.2: now also D52.C, R89.2, T13.2; no longer R99.2
- net T16.4: now also D58.C, R95.2, T13.4; no longer R107.2
- net T9.2: now also D34.C, R54.2; no longer R66.2
- net T9.4: now also D38.C, R62.2; no longer R74.2
- new net N$109: D34.A, R54.1, R66.2
- new net N$119: D38.A, R62.1, R74.2
- new net N$120: D33.A, R53.1, R65.2
- new net N$121: D37.A, R61.1, R73.2
- new net N$122: D32.A, R52.1, R64.2
- new net N$123: D36.A, R60.1, R72.2
- new net N$127: D55.A, R102.2, R92.1
- new net N$135: D61.A, R110.2, R98.1
- new net N$136: D54.A, R101.2, R91.1
- new net N$137: D60.A, R109.2, R97.1
- new net N$138: D53.A, R100.2, R90.1
- new net N$139: D59.A, R108.2, R96.1
- new net N$140: D52.A, R89.1, R99.2
- new net N$141: D58.A, R107.2, R95.1
- new net N$98: D31.A, R51.1, R63.2
- new net N$99: D35.A, R59.1, R71.2
